File: e28_dual_tx/e28_tx.kicad_sch (KiCad schematic)
At the start: 22 parts, among them J1 USB_B_Micro, J2 Conn_01x05, J3 Conn_01x04, J4 Conn_01x04, Q1 BC847BS, SW1 SW_Push, SW2 SW_Push, U1 CH340C, U3 ESP32-WROOM-32D, U4 E28-2G4M27S

Commit message: Last tweaks and gerber files to min_sx1280 and e28_tx
Parts:
- removed H1, H2, H3: MountingHole, MountingHole:MountingHole_3.2mm_M3, symbol Mechanical:MountingHole
- added C10: 10uF, Capacitor_Tantalum_SMD:CP_EIA-1608-08_AVX-J_Pad1.25x1.05mm_HandSolder, symbol device:CP
- added C11: 100nF, Capacitor_SMD:C_0603_1608Metric_Pad1.05x0.95mm_HandSolder, symbol device:C
- added C3, C5: 2.2uF, Capacitor_Tantalum_SMD:CP_EIA-1608-08_AVX-J_Pad1.25x1.05mm_HandSolder, symbol device:CP
- added U2: me6211c33, Package_TO_SOT_SMD:SOT-23-5, symbol regul:TLV70012DDC
- added U5: E28-2G4M27S, ELRS_lib:E28-2G4M27S, symbol ELRS_lib:E28-2G4M27S
- added U?: LoRa1280, symbol ELRS_lib:LoRa1280
- D1: value B5819 -> B5918
Connections:
- net DIO2 is gone; now on net DIO21: U3.24 (IO2), U4.14 (DIO2)
- net +3V3: now also C10.1, C11.1, C5.1, U2.5 (OUT), U5.1 (VCC); no longer J4.4 (Pin_4)
- net BUSY: now also U5.12 (BUSY)
- net GND: now also C10.2, C11.2, C3.2, C5.2, U2.2 (GND), U5.10 (GND), U5.16 (GND), U5.2 (GND), U5.7 (GND)
- net MISO: now also U5.3 (MISO_TX)
- net MOSI: now also U5.4 (MOSI_RX)
- net RESET: now also U5.11 (NRESET)
- net RXEN: now also U5.8 (RX_EN)
- net SCK: now also U5.5 (SCK_RSTN)
- net TXEN: now also U5.9 (TX_EN)
- net VBAT: no longer D1.1 (K)
- net NSS2: now reaches U3.10 (IO25)
- net NSS2: now also U5.6 (NSS_CTS)
- net DIO21: now reaches U3.27 (IO16)
- net DIO12: now reaches U3.28 (IO17)
- net DIO12: now also U5.13 (DIO1)
- net DIO1 renamed DIO11
- net NSS renamed NSS1
- new net +5V: C3.1, D1.1 (K), J4.4 (Pin_4), U2.1 (IN), U2.3 (EN)
- new net DIO22: U5.14 (DIO2)
Other:
- moved on the sheet: C8, C9, J2, J3, J4, U4
